Commit message: controller WIP

File: src/my_legged_robots_sims/urdf/monoped_controlled.urdf (robot description, URDF)
Before this commit: robot monoped, 7 links, 6 joints
Links:
- removed link gantry
- removed link world
- link base: mass 0.4672 -> 10
- link hipassembly: mass 0.1168 -> 0.0292
- link upperleg: mass 0.1168 -> 0.0292
Joints:
- removed joint gantry_to_world
- removed joint vertical_joint
- joint haa_joint: limit lower=-1.0 upper=1.0 effort=200 velocity=3.0 -> lower=-3.14 upper=3.14 effort=1000 velocity=5.0
- joint hfe_joint: limit lower=-1.6 upper=1.6 effort=200 velocity=3.0 -> lower=-3.14 upper=3.14 effort=1000 velocity=5.0
- joint kfe_joint: limit lower=-1.6 upper=0.0 effort=200 velocity=3.0 -> lower=-3.14 upper=3.14 effort=1000 velocity=5.0
